File: antmicro-cvbs-mipi-bridge.kicad_sch (KiCad schematic)
At the start: 65 parts

Commit message: Started converting schematics to antmicro-kicad-library
Parts:
- removed +5V_SYS_2: (no value), symbol power:++5V_SYS
- removed 1.8V: (no value), symbol power:+1.8V
- removed AGPO0, AGPO1, PWR1: (no value), symbol decoder-SchDoc-rescue:LED-
- removed AIN1, AIN2, AIN3, AIN4: (no value), symbol decoder-SchDoc-rescue:CC-134B-
- removed C1, C10, C11, C12, C13, C14, C15, C16, C17, C18, C19, C2, C20, C22, C23, C3, C4, C5, C6, C8, C9: (no value), symbol decoder-SchDoc-rescue:C-
- removed C7: (no value), symbol decoder-SchDoc-rescue:CPol-
- removed IC1: (no value), symbol decoder-SchDoc-rescue:ADV7280-M-
- removed IC2: (no value), symbol decoder-SchDoc-rescue:LP2992AIM5-1.8-
- removed IC3: (no value), symbol decoder-SchDoc-rescue:xx1117-
- removed IC4: (no value), symbol decoder-SchDoc-rescue:SN74LVC1G17-
- removed J7: (no value), symbol decoder-SchDoc-rescue:HEADER_1X2_male-
- removed L1, L2, L3: (no value), symbol decoder-SchDoc-rescue:Inductor_SMT-
- removed Q1: (no value), symbol decoder-SchDoc-rescue:PMGD130UN-
- removed R1, R10, R11, R12, R13, R14, R15, R16, R17, R2, R3, R4, R5, R6, R7, R8, R9: (no value), symbol decoder-SchDoc-rescue:R-
- removed Y1: (no value), symbol decoder-SchDoc-rescue:TXC_7B-
- added AGPO0, AGPO1, PWR1: KP-1608ZGC, antmicro-footprints:LED_0603, symbol antmicroLEDIndicationDiscrete:KP-1608ZGC
- added AIN1, AIN2, AIN3, AIN4: PJRAN1X1U01X, antmicro-footprints:PJRAN1X1U01X, symbol antmicroRCAConnectors:PJRAN1X1U01X
- added C1, C10, C13, C14, C16, C17, C2, C20, C3, C4, C5, C6, C? (x2): C_100n_0402, antmicro-footprints:0402-cap, symbol antmicroCapacitors0402:C_100n_0402
- added C11, C15, C18, C19: C_10n_0402, antmicro-footprints:0402-cap, symbol antmicroCapacitors0402:C_10n_0402
- added C22, C23: C_27p_0402, antmicro-footprints:0402-cap, symbol antmicroCapacitors0402:C_27p_0402
- added C? (x2): C_1u_0402, antmicro-footprints:0402-cap, symbol antmicroCapacitors0402:C_1u_0402
- added C? (x2): C_10u_0402, antmicro-footprints:0402-cap, symbol antmicroCapacitors0402:C_10u_0402
- added FB? (x3): 742792022, antmicro-footprints:0805-res, symbol antmicroFerriteBeadsandChips:742792022
- added IC1: ADV7280BCPZ-M, antmicro-footprints:LFCSP-32-1EP-5x5mm, symbol antmicroDataAcquisitionAnalogtoDigitalConvertersADC:ADV7280BCPZ-M
- added IC2: TLV70018, antmicro-footprints:SC-70-5, symbol antmicroPMICVoltageRegulatorsLinear:TLV70018
- added IC3: NCP1117ST33T3G, antmicro-footprints:SOT-223, symbol antmicroPMICVoltageRegulatorsLinear:NCP1117ST33T3G
- added IC4: SN74AUP1G17DCKR, antmicro-footprints:SOT-753, symbol antmicroLogicBuffersDriversReceiversTransceivers:SN74AUP1G17DCKR
- added J7: 61300211121, antmicro-footprints:PinHeader_1x2_P2.54_Drill0.9mm, symbol antmicroRectangularConnectorsHeadersMalePins:61300211121
- added Q1: NX3008NBKS_2, antmicro-footprints:SOT-363, symbol antmicroTransistorsFETsMOSFETsArrays:NX3008NBKS_2
- added R1, R10, R4, R8: R_24R_0603, antmicro-footprints:0603-res, symbol antmicroResistors0603:R_24R_0603
- added R11, R3, R5, R9: R_51R_0402, antmicro-footprints:0402-res, symbol antmicroResistors0402:R_51R_0402
- added R12, R13, R14: R_330R_0402, antmicro-footprints:0402-res, symbol antmicroResistors0402:R_330R_0402
- added R15: R_22k_0402, antmicro-footprints:0402-res, symbol antmicroResistors0402:R_22k_0402
- added R16: R_1M0_0402, antmicro-footprints:0402-res, symbol antmicroResistors0402:R_1M0_0402
- added R2: R_1k_0402, antmicro-footprints:0402-res, symbol antmicroResistors0402:R_1k_0402
- added R6, R7: R_4k7_0402, antmicro-footprints:0402-res, symbol antmicroResistors0402:R_4k7_0402
- added R? (x2): R_0R_0402, antmicro-footprints:0402-res, symbol antmicroResistors0402:R_0R_0402
- added R?: R_100k_0402, antmicro-footprints:0402-res, symbol antmicroResistors0402:R_100k_0402
- added Y1: ABM8G-28.63636MHZ-18-D2Y-T, antmicro-footprints:KX-7, symbol antmicroCrystals:ABM8G-28.63636MHZ-18-D2Y-T
- +5V_SYS, C21, C24, IC5, J1, R18, R19: value (none) -> ~
Connections:
- net +3V3: now also IC1.28 (~{RESET})
- net AGPO0: now also IC1.8 (GPO0), Q1.2 (G1)
- net AGPO1: now also IC1.7 (GPO1), Q1.5 (G2)
- net AIN1: now also C1.2, IC1.17 (AIN1)
- net AIN2: now also C2.2, IC1.18 (AIN2)
- net AIN3: now also C4.2, IC1.22 (AIN3)
- net AIN4: now also C10.2, IC1.23 (AIN4)
- net CSI_A_CLK_N: now also IC1.12 (CLK_N); no longer J1.1, J1.7, J1.8
- net GND: now also AIN1.1, AIN1.3, AIN2.1, AIN2.3, AIN3.1, AIN3.3, AIN4.1, AIN4.3, C11.2, C13.2, C14.1, C15.2, C16.1, C17.1, C18.2, C19.2, C20.2, C22.2, C23.2, C3.1, C5.1, C?.1, C?.1, C?.2, C?.2, C?.2, C?.2, IC1.1 (DGND), IC1.33 (EP), IC1.4 (DGND), IC2.2 (GND), IC3.1 (ADJ/GND), IC4.3 (GND), J7.2, PWR1.2, Q1.1 (S1), Q1.4 (S2), R11.1, R3.1, R5.1, R9.1, Y1.2, Y1.4
- net SCL: now also IC1.31 (SCLK), R7.1
- net SDA: now also IC1.30 (SDATA), R6.1
- new net: C13.1, IC4.2 (A), R15.1
- new net: C10.1, R10.2, R11.2
- new net: AGPO0.1, R12.2
- new net: AGPO0.2, Q1.6 (D1)
- new net: PWR1.1, R14.2
- new net: AIN4.2, R10.1
- new net: C?.1, IC3.2 (OUT), IC3.4 (OUT), R?.1
- new net: AGPO1.2, Q1.3 (D2)
- new net: AIN3.2, R8.1
- new net: C?.1, IC2.5 (VOUT), R?.1
- new net: C4.1, R8.2, R9.2
- new net: AIN2.2, R4.1
- new net: C2.1, R4.2, R5.2
- new net: AGPO1.1, R13.1
- new net: C1.1, R1.2, R3.2
- new net: AIN1.2, R1.1
- new net 1V8_SYS: C?.2, FB?.1, FB?.1, FB?.1, R?.2
- new net 3V3_SYS: C20.1, C5.2, C?.1, C?.2, IC1.2 (DVDDIO), IC2.1 (VIN), IC2.3 (EN), IC4.5 (VCC), R12.1, R13.2, R14.1, R15.2, R2.1, R6.2, R7.2, R?.2, R?.2
- new net 5V_SYS: C?.1, IC3.3 (IN)
- new net ALSB: IC1.29 (ALSB), J7.1, R2.2
- new net AVDD_1V8: C14.2, C15.1, FB?.2, IC1.16 (PVDD)
- new net CSI_A_CLK_P: IC1.11 (CLK_P), J1.1
- new net CSI_A_D0_N: IC1.10 (D0_N), J1.7
- new net CSI_A_D0_P: IC1.9 (D0_P), J1.8
- new net DVDD_1V8: C16.2, C17.2, C18.1, C19.1, FB?.2, IC1.13 (MVDD), IC1.3 (DVDD)
- new net PVDD_1V8: C11.1, C3.2, FB?.2, IC1.21 (AVDD)
- new net PWRDWN: IC1.32 (~{PWRDWN}), IC4.4 (Y), R?.1
- new net VREFN: C6.1, IC1.20 (VREFN)
- new net VREFP: C6.2, IC1.19 (VREFP)
- new net XTAL_N: C22.1, IC1.15 (XTALN), R16.1, Y1.1
- new net XTAL_P: C23.1, IC1.14 (XTALP), R16.2, Y1.3
Other:
- note added: "50-pin FFC Connector"
- note added: "Decoupling"
- note added: "LED Indicators"
- note added: "Power Supply"
- note added: "RCA Connectors"
- note added: "RCA to MIPI decoder"
- moved on the sheet: C21, C24, IC5, J1, R18, R19

Commit message: Finished correcting schematics
Parts:
- removed +5V_SYS: ~, symbol power:++5V_SYS
- removed C21, C24: ~, symbol decoder-SchDoc-rescue:C-
- removed C22, C23: C_27p_0402, antmicro-footprints:0402-cap, symbol antmicroCapacitors0402:C_27p_0402
- removed C? (x2): C_10u_0402, antmicro-footprints:0402-cap, symbol antmicroCapacitors0402:C_10u_0402
- removed IC3: NCP1117ST33T3G, antmicro-footprints:SOT-223, symbol antmicroPMICVoltageRegulatorsLinear:NCP1117ST33T3G
- removed IC5: ~, symbol decoder-SchDoc-rescue:SN74LVC1G17-
- removed J1: ~, symbol decoder-SchDoc-rescue:RJ45_AMP-1-406541-
- removed R12, R13, R14: R_330R_0402, antmicro-footprints:0402-res, symbol antmicroResistors0402:R_330R_0402
- removed R18, R19: ~, symbol decoder-SchDoc-rescue:R-
- removed R?: R_0R_0402, antmicro-footprints:0402-res, symbol antmicroResistors0402:R_0R_0402
- added C12, C25: C_1u_0603, antmicro-jetson-agx-csi-adapter-footprints:0603-cap, symbol antmicro-jetson-agx-csi-adapter:C_1u_0603
- added C21, C24: C_100n_0402, antmicro-footprints:0402-cap, symbol antmicroCapacitors0402:C_100n_0402
- added C22, C23: C_10p_0402, antmicro-footprints:0402-cap, symbol antmicroCapacitors0402:C_10p_0402
- added C27, C28: C_1u_0402, antmicro-footprints:0402-cap, symbol antmicroCapacitors0402:C_1u_0402
- added D1, D2, D3, D4: PESD1CAN_215, antmicro-footprints:SOT-23-3, symbol antmicroTVSDiodes:PESD1CAN_215
- added FB1, FB2: 742792022, antmicro-footprints:0805-res, symbol antmicroFerriteBeadsandChips:742792022
- added IC5: SN74AUP1G17DCKR, antmicro-footprints:SOT-753, symbol antmicroLogicBuffersDriversReceiversTransceivers:SN74AUP1G17DCKR
- added J1: WE_68715014522_ONE-SIDE, antmicro-jetson-agx-csi-adapter-footprints:WE_68715014522_ONE-SIDE, symbol antmicro-jetson-agx-csi-adapter:WE_68715014522_ONE-SIDE
- added J2: 61300211121, antmicro-footprints:PinHeader_1x2_P2.54_Drill0.9mm, symbol antmicroRectangularConnectorsHeadersMalePins:61300211121
- added PWR1, PWR3: KP-1608ZGC, antmicro-footprints:LED_0603, symbol antmicroLEDIndicationDiscrete:KP-1608ZGC
- added Q2: BSS138APW, antmicro-footprints:SC70-3, symbol antmicroTransistorsFETsMOSFETsSingle:BSS138APW
- added R12, R13, R14, R26: R_470R_0402, antmicro-jetson-agx-csi-adapter-footprints:0402-res, symbol antmicro-jetson-agx-csi-adapter:R_470R_0402
- added R18, R19, R28: R_100k_0402, antmicro-footprints:0402-res, symbol antmicroResistors0402:R_100k_0402
- added R20, R21, R22, R23, R24, R25: R_0R_0402, antmicro-footprints:0402-res, symbol antmicroResistors0402:R_0R_0402
- added R27, R29: R_1k_0402, antmicro-footprints:0402-res, symbol antmicroResistors0402:R_1k_0402
- added S1: KMR2, antmicro-footprints:SW_SPST_4.2x2.8, symbol antmicroPushbuttonSwitches:KMR2
- added TP1, TP10, TP11, TP12, TP13, TP2, TP3, TP4, TP5, TP6, TP7, TP8, TP9: TP, antmicro-footprints:TP-R-1.5, symbol antmicroTestPoints:TP
- gave numbers to parts that had none: 9
- renumbered PWR1 to PWR2
Connections:
- net 1V8_SYS: now also Q2.1 (G), R28.2
- net 3V3_SYS: now also C24.1, C27.1, C28.1, FB1.1, IC5.5 (VCC), J2.2, R12.2, R13.2, R14.1, R18.2, R19.2, R26.1, TP5.1
- net 5V_SYS: now also FB2.1, R27.1, TP4.1
- net AGPO0: now also TP11.1
- net AGPO1: now also TP10.1
- net ALSB: now also TP12.1
- net CSI_A_CLK_N: now also R24.1
- net CSI_A_CLK_P: now also R25.1
- net CSI_A_D0_N: now also R22.1
- net CSI_A_D0_P: now also R23.1
- net GND: now also C12.2, C21.2, C22.2, C23.2, C24.2, C25.2, C27.2, C28.2, D1.3 (C3), D2.3 (C3), D3.3 (C3), D4.3 (C3), IC5.3 (GND), J1.12 (Pin_12), J1.15 (Pin_15), J1.18 (Pin_18), J1.27 (Pin_27), J1.30 (Pin_30), J1.9 (Pin_9), J2.1, PWR1.2, Q2.2 (S), R28.1, S1.1, S1.3, TP13.1
- net PWRDWN: now also TP9.1
- net RST_IN: now also J1.33 (Pin_33), R29.1
- net SCL: now also R21.1, TP7.1
- net SDA: now also R20.1, TP6.1
- net XTAL_N: now also C22.1
- net XTAL_P: now also C23.1
- net at AGPO0.1: now also R12.1
- net at PWR2.1: now also R14.2
- net AIN4_ESD: now reaches AIN4.2, R10.1
- net AIN4_ESD: now also D4.1 (C1)
- net AIN3_ESD: now reaches AIN3.2, R8.1
- net AIN3_ESD: now also D3.1 (C1)
- net at C9.1, IC2.5 (VOUT), R30.1: now also TP3.1
- net AIN2_ESD: now reaches AIN2.2, R4.1
- net AIN2_ESD: now also D2.1 (C1)
- net at AGPO1.1: now also R13.1
- net at IC1.5 (~{INTRQ}): now also TP2.1
- net at IC1.6 (GPO2): now also TP1.1
- net AIN1_ESD: now reaches AIN1.2, R1.1
- net AIN1_ESD: now also D1.1 (C1)
- net +3V3 renamed RESET
- net RESET: now also IC5.4 (Y), R19.1, TP8.1
- new net: J1.25 (Pin_25), R22.2
- new net: J1.26 (Pin_26), R23.2
- new net: J1.28 (Pin_28), R24.2
- new net: J1.29 (Pin_29), R25.2
- new net: J1.39 (Pin_39), R20.2
- new net: J1.40 (Pin_40), R21.2
- new net: C12.1, FB1.2, J1.47 (Pin_47), J1.48 (Pin_48)
- new net: C25.1, FB2.2, J1.49 (Pin_49), J1.50 (Pin_50)
- new net: C21.1, IC5.2 (A), R18.1, R29.2, S1.2, S1.4
- new net: PWR1.1, R27.2
- new net: PWR3.1, R26.2
- new net: PWR3.2, Q2.3 (D)
- no-connect marks 6 -> 41
Other:
- note added: "CSI"
- note added: "Control interface"
- note added: "Debug Power Supply Connector"
- note added: "Power On Delay"
- note added: "Test points"
- note added: "info: impedance 75R"
- moved on the sheet: AGPO0, AGPO1, AIN1, AIN2, AIN3, AIN4, C1, C10, C11, C13, C14, C15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

Commit message: Reordered components on schematic. Bumped revision to 1.2.0
Other:
- note added: "ADV7280-M Decoupling"
- note added: "RCA ESD"
- note removed: "Decoupling"
- moved on the sheet: AGPO0, AGPO1, AIN1, AIN2, AIN3, AIN4, C1, C10, C11, C12, C13, C14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

Commit message: Started component positions adjusment and placement
Parts:
- added MP1, MP2, MP3, MP4: 9774030243R, antmicro-footprints:9774030243R, symbol antmicroMechanicalParts:9774030243R
- added N1: antmicro_logo, antmicro-footprints:antmicro-logo_scaled_20mm, symbol antmicroMechanicalParts:antmicro_logo
- added N2: oshw_logo, antmicro-footprints:oshw-logo, symbol antmicroMechanicalParts:oshw_logo
- C12, C25: footprint antmicro-jetson-agx-csi-adapter-footprints:0603-cap -> antmicro-footprints:0603-cap
- J1: footprint antmicro-jetson-agx-csi-adapter-footprints:WE_68715014522_ONE-SIDE -> antmicro-footprints:WE_68715014522_ONE-SIDE
- R12, R13, R14, R26: footprint antmicro-jetson-agx-csi-adapter-footprints:0402-res -> antmicro-footprints:0402-res
Other:
- note added: "MISC"
