File: cvbs-mipi-bridge.kicad_pcb (KiCad board)
At the start: 4 copper layers, 55 x 70 mm, 114 parts, among them IC1 ADV7282-M, IC2 TLV70018, IC4 SN74AUP1G17DCKR, IC5 SN74AUP1G17DCKR, J1 WE_68715014522, J2 1053131102, J3 KLPX-0848A-2-Y, J4 KLPX-0848A-2-Y, J5 KLPX-0848A-2-Y, J6 KLPX-0848A-2-Y, J7 61300211121, Q1 BSS138PW, Q2 BSS138PW, Q3 BSS138PW, Q4 BSS138PW, Y1 ABM8G-28.63636MHZ-18-D2Y-T

Commit message: Add connectors & button descriptions to B.Silkscreen
Other:
- board text added: "FFC-50 MIPI CSI-2 Connector"
- board text added: "J7"
- board text added: "RESET"
- board text added: "S1"
Changed lines of the file:
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@@
     )
   )
+  (gr_line (start 155.5 59.7) (end 155.5 56.4) (layer "B.SilkS") (width 0.15))
+  (gr_line (start 130.5 59.7) (end 130.5 56.4) (layer "B.SilkS") (width 0.15))
   (gr_line (start 131.85 92.2) (end 132.1 92.45) (layer "F.SilkS") (width 0.15))
   (gr_circle (center 157.2 88.4) (end 157.4 88.4) (layer "F.SilkS") (width 0.15) (fill none))
@@
   (gr_line (start 111.7 56) (end 166.7 56) (layer "Edge.Cuts") (width 0.254))
   (gr_line (start 111.7 126) (end 166.7 126) (layer "Edge.Cuts") (width 0.254))
+  (gr_text "S1" (at 163 93.5 90) (layer "B.SilkS")
+    (effects (font (size 1 1) (thickness 0.15)) (justify mirror))
+  )
+  (gr_text "J7" (at 156.1 80.6 90) (layer "B.SilkS")
+    (effects (font (size 1 1) (thickness 0.15)) (justify mirror))
+  )
+  (gr_text "AnalogIn4" (at 118.25 112.25 90) (layer "B.SilkS")
+    (effects (font (size 1 1) (thickness 0.15)) (justify mirror))
+  )
+  (gr_text "AnalogIn2\n" (at 118.25 84.200001 90) (layer "B.SilkS")
+    (effects (font (size 1 1) (thickness 0.15)) (justify mirror))
+  )
+  (gr_text "RESET" (at 160.8 93.5 90) (layer "B.SilkS")
+    (effects (font (size 1 1) (thickness 0.15)) (justify mirror))
+  )
+  (gr_text "FFC-50 MIPI CSI-2 Connector" (at 142.9 58) (layer "B.SilkS")
+    (effects (font (size 1 1) (thickness 0.15)) (justify mirror))
+  )
+  (gr_text "AnalogIn3" (at 118.25 98.25 90) (layer "B.SilkS")
+    (effects (font (size 1 1) (thickness 0.15)) (justify mirror))
+  )
+  (gr_text "AnalogIn1" (at 118.25 70.350001 90) (layer "B.SilkS")
+    (effects (font (size 1 1) (thickness 0.15)) (justify mirror))
+  )
+  (gr_text "DebugPower\n3V3" (at 118.25 122.75 90) (layer "B.SilkS")
+    (effects (font (size 0.65 0.65) (thickness 0.15)) (justify mirror))
+  )
   (gr_text "AGPO2" (at 159.3 79.85 90) (layer "F.SilkS")
     (effects (font (size 0.65 0.65) (thickness 0.15)) (justify left))

Commit message: Update PCB nets from SCH
Connections:
- net Net-(IC1-Pad5) renamed /~{INTRQ}
- net Net-(IC1-Pad6) renamed /AGPO2
Changed lines of the file:
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@@
   (net 22 "/XTAL_P")
   (net 23 "1V8_SYS")
-  (net 24 "Net-(IC1-Pad5)")
-  (net 25 "Net-(IC1-Pad6)")
+  (net 24 "/~{INTRQ}")
+  (net 25 "/AGPO2")
   (net 26 "/AGPO1")
   (net 27 "/AGPO0")
@@
       (net 3 "GND") (pinfunction "DGND") (pintype "unspecified"))
     (pad "5" smd rect (at -2.4511 0.25 270) (size 0.254 0.8128) (layers "F.Cu" "F.Paste" "F.Mask")
-      (net 24 "Net-(IC1-Pad5)") (pinfunction "~{INTRQ}") (pintype "output"))
+      (net 24 "/~{INTRQ}") (pinfunction "~{INTRQ}") (pintype "output"))
     (pad "6" smd rect (at -2.4511 0.750001 270) (size 0.254 0.8128) (layers "F.Cu" "F.Paste" "F.Mask")
-      (net 25 "Net-(IC1-Pad6)") (pinfunction "GPO2") (pintype "bidirectional"))
+      (net 25 "/AGPO2") (pinfunction "GPO2") (pintype "bidirectional"))
     (pad "7" smd rect (at -2.4511 1.25 270) (size 0.254 0.8128) (layers "F.Cu" "F.Paste" "F.Mask")
       (net 26 "/AGPO1") (pinfunction "GPO1") (pintype "bidirectional"))
@@
     )
     (pad "1" smd circle locked (at 0 0 270) (size 1.5 1.5) (layers "F.Cu" "F.Mask")
-      (net 25 "Net-(IC1-Pad6)") (pintype "passive"))
+      (net 25 "/AGPO2") (pintype "passive"))
   )
   (footprint "cvbs-mipi-bridge-footprints:TP-R-1.5" (layer "F.Cu")
@@
     )
     (pad "1" smd circle locked (at 0 0 90) (size 1.5 1.5) (layers "F.Cu" "F.Mask")
-      (net 24 "Net-(IC1-Pad5)") (pintype "passive"))
+      (net 24 "/~{INTRQ}") (pintype "passive"))
   )
   (footprint "cvbs-mipi-bridge-footprints:0402-cap" (layer "F.Cu")

Commit message: Update antmicro_logo footprint reference to correct one
Update in local library, then on SCH, then updated PCB from SCH
Parts:
- N1: footprint cvbs-mipi-bridge-footprints:antmicro-logo_scaled_20mm -> antmicro-footprints:antmicro-logo_scaled_20mm_mask
