File: cvbs-mipi-bridge.kicad_sch (KiCad schematic)
At the start: 114 parts, among them IC1 ADV7282-M, IC2 TLV70018_SC70, IC4 SN74AUP1G17_SC70, IC5 SN74AUP1G17_SC70, J1 Conn_FFC_WE_68715014522, J2 Molex_Nano-Fit_1x2_1053131102, J3 RCA_Jack_KLPX-0848A-2-Y, J4 RCA_Jack_KLPX-0848A-2-Y, J5 RCA_Jack_KLPX-0848A-2-Y, J6 RCA_Jack_KLPX-0848A-2-Y, J7 PinHeader_1x2_P2.54mm_Drill1.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, Q1 BSS138PW, Q2 BSS138PW, Q3 BSS138PW, Q4 BSS138PW, Y1 Resonator_28.63636MHz_ABM8G

Commit message: [#56797] Loclib
Parts:
- C1, C10, C13, C14, C16, C17, C2, C20, C21, C24, C26, C29, C3, C4, C5, C6, C7: footprint antmicro-footprints:C_0402_1005Metric -> cvbs-mipi-bridge-footprints:C_0402_1005Metric; symbol antmicroCapacitors0402:C_100n_0402 -> cvbs-mipi-bridge:C_100n_0402
- C11, C15, C18, C19: footprint antmicro-footprints:C_0402_1005Metric -> cvbs-mipi-bridge-footprints:C_0402_1005Metric; symbol antmicroCapacitors0402:C_10n_0402 -> cvbs-mipi-bridge:C_10n_0402
- C12: footprint antmicro-footprints:C_0603_1608Metric -> cvbs-mipi-bridge-footprints:C_0603_1608Metric; symbol antmicroCapacitors0603:C_1u_0603 -> cvbs-mipi-bridge:C_1u_0603
- C22, C23: footprint antmicro-footprints:C_0402_1005Metric -> cvbs-mipi-bridge-footprints:C_0402_1005Metric; symbol antmicroCapacitors0402:C_10p_0402 -> cvbs-mipi-bridge:C_10p_0402
- C25, C27, C28, C8, C9: footprint antmicro-footprints:C_0402_1005Metric -> cvbs-mipi-bridge-footprints:C_0402_1005Metric; symbol antmicroCapacitors0402:C_1u_0402 -> cvbs-mipi-bridge:C_1u_0402
- C30, C31, C32: footprint antmicro-footprints:C_0603_1608Metric -> cvbs-mipi-bridge-footprints:C_0603_1608Metric; symbol antmicroCapacitors0603:C_10u_0603 -> cvbs-mipi-bridge:C_10u_0603
- D1, D2, D3, D4: footprint antmicro-footprints:SLP1006P2T -> cvbs-mipi-bridge-footprints:SLP1006P2T; symbol antmicroTVSDiodes:UCLAMP2501T.TCT -> cvbs-mipi-bridge:UCLAMP2501T.TCT
- D5, D6, D7, D8: footprint antmicro-footprints:LED_0603_1608Metric_G -> cvbs-mipi-bridge-footprints:LED_0603_1608Metric_G; symbol antmicroLEDIndicationDiscrete:LED_G_0603_KP-1608ZGC -> cvbs-mipi-bridge:LED_G_0603_KP-1608ZGC
- FB1, FB3, FB4, FB5: footprint antmicro-footprints:FB_0805_2012Metric -> cvbs-mipi-bridge-footprints:FB_0805_2012Metric; symbol antmicroFerriteBeadsandChips:FB_220Z_1.5A_WE-CBF_0805 -> cvbs-mipi-bridge:FB_220Z_1.5A_WE-CBF_0805
- IC1: footprint antmicro-footprints:LFCSP-32-1EP-5x5mm -> cvbs-mipi-bridge-footprints:LFCSP-32-1EP-5x5mm; symbol antmicroDataAcquisitionAnalogtoDigitalConvertersADC:ADV7282-M -> cvbs-mipi-bridge:ADV7282-M
- IC2: footprint antmicro-footprints:SC-70-5 -> cvbs-mipi-bridge-footprints:SC-70-5; symbol antmicroPMICVoltageRegulatorsLinear:TLV70018_SC70 -> cvbs-mipi-bridge:TLV70018_SC70
- IC4, IC5: footprint antmicro-footprints:SC-70-5 -> cvbs-mipi-bridge-footprints:SC-70-5; symbol antmicroLogicBuffersDriversReceiversTransceivers:SN74AUP1G17_SC70 -> cvbs-mipi-bridge:SN74AUP1G17_SC70
- J1: footprint antmicro-footprints:Conn_FFC_WE_68715014x22 -> cvbs-mipi-bridge-footprints:Conn_FFC_WE_68715014x22; symbol antmicroFCCConnectors:Conn_FFC_WE_68715014522 -> cvbs-mipi-bridge:Conn_FFC_WE_68715014522
- J2: footprint antmicro-footprints:Conn_Molex_Nano-Fit_1x2_1053131102 -> cvbs-mipi-bridge-footprints:Conn_Molex_Nano-Fit_1x2_1053131102; symbol antmicroWire2BoardConnectors:Molex_Nano-Fit_1x2_1053131102 -> cvbs-mipi-bridge:Molex_Nano-Fit_1x2_1053131102
- J3, J4, J5, J6: footprint antmicro-footprints:RCA_Jack_KLPX-0848A-2-Y -> cvbs-mipi-bridge-footprints:RCA_Jack_KLPX-0848A-2-Y; symbol antmicroBarrelAudioConnectors:RCA_Jack_KLPX-0848A-2-Y -> cvbs-mipi-bridge:RCA_Jack_KLPX-0848A-2-Y
- J7: footprint antmicro-footprints:PinHeader_1x2_P2.54_Drill0.9mm -> cvbs-mipi-bridge-footprints:PinHeader_1x2_P2.54_Drill0.9mm; symbol antmicroGenericPinHeaders:PinHeader_1x2_P2.54mm_Drill1.1mm -> cvbs-mipi-bridge:PinHeader_1x2_P2.54mm_Drill1.1mm
- MP1, MP2, MP3, MP4: footprint antmicro-footprints:Spacer_Drill3mm_H3mm_9774030243R -> cvbs-mipi-bridge-footprints:Spacer_Drill3mm_H3mm_9774030243R; symbol antmicroMechanicalParts:Spacer_Drill3mm_H3mm_9774030243R -> cvbs-mipi-bridge:Spacer_Drill3mm_H3mm_9774030243R
- Q1, Q2, Q3, Q4: footprint antmicro-footprints:SC70-3 -> cvbs-mipi-bridge-footprints:SC70-3; symbol antmicroTransistorsFETsMOSFETsSingle:BSS138PW -> cvbs-mipi-bridge:BSS138PW
- R1, R10, R4, R8: footprint antmicro-footprints:R_0402_1005Metric -> cvbs-mipi-bridge-footprints:R_0402_1005Metric; symbol antmicroResistors0402:R_24R_0402 -> cvbs-mipi-bridge:R_24R_0402
- R11, R3, R5, R9: footprint antmicro-footprints:R_0402_1005Metric -> cvbs-mipi-bridge-footprints:R_0402_1005Metric; symbol antmicroResistors0402:R_51R_0402 -> cvbs-mipi-bridge:R_51R_0402
- R12, R13, R14, R26: footprint antmicro-footprints:R_0402_1005Metric -> cvbs-mipi-bridge-footprints:R_0402_1005Metric; symbol antmicroResistors0402:R_470R_0402 -> cvbs-mipi-bridge:R_470R_0402
- R15: footprint antmicro-footprints:R_0402_1005Metric -> cvbs-mipi-bridge-footprints:R_0402_1005Metric; symbol antmicroResistors0402:R_22k_0402 -> cvbs-mipi-bridge:R_22k_0402
- R16: footprint antmicro-footprints:R_0402_1005Metric -> cvbs-mipi-bridge-footprints:R_0402_1005Metric; symbol antmicroResistors0402:R_1M_0402 -> cvbs-mipi-bridge:R_1M_0402
- R17, R18, R19, R27, R28, R29, R31: footprint antmicro-footprints:R_0402_1005Metric -> cvbs-mipi-bridge-footprints:R_0402_1005Metric; symbol antmicroResistors0402:R_100k_0402 -> cvbs-mipi-bridge:R_100k_0402
- R2: footprint antmicro-footprints:R_0402_1005Metric -> cvbs-mipi-bridge-footprints:R_0402_1005Metric; symbol antmicroResistors0402:R_1k_0402 -> cvbs-mipi-bridge:R_1k_0402
- R20, R21, R22, R23, R24, R25, R32, R33: footprint antmicro-footprints:R_0402_1005Metric -> cvbs-mipi-bridge-footprints:R_0402_1005Metric; symbol antmicroResistors0402:R_0R_0402 -> cvbs-mipi-bridge:R_0R_0402
- R30: footprint antmicro-footprints:R_0805_2012Metric -> cvbs-mipi-bridge-footprints:R_0805_2012Metric; symbol antmicroResistorsmisc:R_0R_0805 -> cvbs-mipi-bridge:R_0R_0805
- R6, R7: footprint antmicro-footprints:R_0402_1005Metric -> cvbs-mipi-bridge-footprints:R_0402_1005Metric; symbol antmicroResistors0402:R_4k7_0402 -> cvbs-mipi-bridge:R_4k7_0402
- S1: footprint antmicro-footprints:SW_KMR211NGLFS_SMD -> cvbs-mipi-bridge-footprints:SW_KMR211NGLFS_SMD; symbol antmicroPushbuttonSwitches:SW_KMR211NGLFS_SMD -> cvbs-mipi-bridge:SW_KMR211NGLFS_SMD
- TP1, TP10, TP11, TP12, TP13, TP14, TP15, TP16, TP2, TP3, TP4, TP5, TP6, TP7, TP8, TP9: footprint antmicro-footprints:TP_SMD_1.5mm -> cvbs-mipi-bridge-footprints:TP_SMD_1.5mm; symbol antmicroTestPoints:TP_1.5mm_SMD -> cvbs-mipi-bridge:TP_1.5mm_SMD
- Y1: footprint antmicro-footprints:Oscillator_SMD_Geyer_KX-7-4Pin_3.2x2.5mm -> cvbs-mipi-bridge-footprints:Oscillator_SMD_Geyer_KX-7-4Pin_3.2x2.5mm; symbol antmicroResonators:Resonator_28.63636MHz_ABM8G -> cvbs-mipi-bridge:Resonator_28.63636MHz_ABM8G
